Commit message: Added Rune's Kuka modifications

File: kuka_kr10_support/urdf/kr10r1100sixx_macro.xacro (robot description, xacro)
@@ -8,5 +8,5 @@
         <origin xyz="0 0 0" rpy="0 0 0"/>
         <geometry>
-          <mesh filename="package://kuka_kr10_support/meshes/kr10r1100sixx/visual/base_link.stl" />
+          <mesh filename="package://kuka_kr10_support/meshes/kr10r1100sixx/visual/base.stl" />
         </geometry>
         <xacro:material_kuka_black />
@@ -15,5 +15,5 @@
         <origin xyz="0 0 0" rpy="0 0 0"/>
         <geometry>
-          <mesh filename="package://kuka_kr10_support/meshes/kr10r1100sixx/collision/base_link.stl" />
+          <mesh filename="package://kuka_kr10_support/meshes/kr10r1100sixx/collision/base.stl" />
         </geometry>
       </collision>

File: kuka_resources/urdf/common_colours.xacro (robot description, xacro)
@@ -72,5 +72,3 @@
   <!-- RAL 9002 - gray white  -->
   <xacro:property name="colour_kuka_ral_gray_white"       value="${215/255} ${213/255} ${203/255} 1.0" />
-  <!-- RAL 9010 - pure white  -->
-  <xacro:property name="colour_kuka_ral_pure_white"       value="${241/255} ${236/255} ${255/255} 1.0" />
 </robot>

File: kuka_resources/urdf/common_materials.xacro (robot description, xacro)
@@ -152,8 +152,3 @@
     </material>
   </xacro:macro>
-  <xacro:macro name="material_kuka_ral_pure_white">
-    <material name="">
-      <color rgba="${colour_kuka_ral_pure_white}"/>
-    </material>
-  </xacro:macro>
 </robot>
